File: PCB-kicad/ibutton.sch (KiCad schematic (older format))
At the start: 30 parts, among them J1 I_BUTTON, J2 IB_READ, J3 BATTERY, J4 USB_OTG, Q1 BC847, Q2 BC847, SW1 SW_Push, U1 ATMEGA8-16AU, U2 CH340G, Y1 12MHz

Commit message: разработка печатной платы
Parts:
- C1, C2, C3: footprint Capacitors_THT:CP_Radial_D5.0mm_P2.50mm -> Capacitor_SMD:C_0805_2012Metric_Pad1.15x1.40mm_HandSolder
- C4, C5, C6: footprint (none) -> Capacitor_SMD:C_0805_2012Metric_Pad1.15x1.40mm_HandSolder
- D1, D2: footprint Diodes_SMD:D_SOT-23_NKA -> Diode_SMD:D_SOT-23_NKA
- D3, D5: footprint (none) -> LED_THT:LED_D5.0mm
- D4: value 2^3 -> 2^2; footprint (none) -> LED_THT:LED_D5.0mm
- D6: value 2^4 -> 2^3; footprint (none) -> LED_THT:LED_D5.0mm
- J1, J2: footprint Connectors_Molex:Molex_MicroLatch-53253-0270_02x2.00mm_Straight -> Connector_PinHeader_2.54mm:PinHeader_1x02_P2.54mm_Vertical
- J3: footprint Connectors:bornier2 -> Connector_PinHeader_2.54mm:PinHeader_1x02_P2.54mm_Vertical
- J4: footprint Connectors:USB_Mini-B -> Connector_USB:USB_Micro-B_Wuerth_629105150521
- Q1, Q2: footprint TO_SOT_Packages_SMD:SOT-23 -> Package_TO_SOT_SMD:SOT-23_Handsoldering
- R1, R2, R4, R5, R7: footprint Resistors_SMD:R_0402_NoSilk -> Resistor_SMD:R_0805_2012Metric_Pad1.15x1.40mm_HandSolder
- R3, R6, R8: footprint Resistors_THT:R_Axial_DIN0204_L3.6mm_D1.6mm_P7.62mm_Horizontal -> Resistor_SMD:R_0805_2012Metric_Pad1.15x1.40mm_HandSolder
- SW1: footprint Buttons_Switches_SMD:SW_SPST_PTS645 -> Button_Switch_SMD:SW_SPST_PTS645
- U1: footprint Housings_QFP:TQFP-32_7x7mm_Pitch0.8mm -> Package_DIP:DIP-32_W7.62mm
- Y1: footprint (none) -> Crystal:Crystal_SMD_HC49-SD
Connections:
- net at U1.13 ((OC1A)PB1): now also D6.2 (A); no longer D3.2 (A)
- net at U1.14 ((~SS~/OC1B)PB2): now also D4.2 (A); no longer D5.2 (A)
- net at U1.15 ((MOSI/OC2)PB3): now also D5.2 (A); no longer D4.2 (A)
- net at U1.16 ((MISO)PB4): now also D3.2 (A); no longer D6.2 (A)
- no-connect marks 8 -> 21
Changed lines of the file:
@@
 F 0 "R5" V 6530 4150 40  0000 C CNN
 F 1 "100K" V 6457 4151 40  0000 C CNN
-F 2 "Resistors_SMD:R_0402_NoSilk" V 6380 4150 30  0001 C CNN
+F 2 "Resistor_SMD:R_0805_2012Metric_Pad1.15x1.40mm_HandSolder" V 6380 4150 30  0001 C CNN
 F 3 "~" H 6450 4150 30  0000 C CNN
 	1    6450 4150
@@
 F 0 "R4" V 5830 4150 40  0000 C CNN
 F 1 "5K" V 5757 4151 40  0000 C CNN
-F 2 "Resistors_SMD:R_0402_NoSilk" V 5680 4150 30  0001 C CNN
+F 2 "Resistor_SMD:R_0805_2012Metric_Pad1.15x1.40mm_HandSolder" V 5680 4150 30  0001 C CNN
 F 3 "~" H 5750 4150 30  0000 C CNN
 	1    5750 4150
@@
 F 0 "R8" V 7930 3100 40  0000 C CNN
 F 1 "5K" V 7857 3101 40  0000 C CNN
-F 2 "Resistors_THT:R_Axial_DIN0204_L3.6mm_D1.6mm_P7.62mm_Horizontal" V 7780 3100 30  0001 C CNN
+F 2 "Resistor_SMD:R_0805_2012Metric_Pad1.15x1.40mm_HandSolder" V 7780 3100 30  0001 C CNN
 F 3 "~" H 7850 3100 30  0000 C CNN
 	1    7850 3100
@@
 F 0 "R7" V 7930 2450 40  0000 C CNN
 F 1 "5K" V 7857 2451 40  0000 C CNN
-F 2 "Resistors_SMD:R_0402_NoSilk" V 7780 2450 30  0001 C CNN
+F 2 "Resistor_SMD:R_0805_2012Metric_Pad1.15x1.40mm_HandSolder" V 7780 2450 30  0001 C CNN
 F 3 "~" H 7850 2450 30  0000 C CNN
 	1    7850 2450
@@
 F 0 "R2" V 3680 2300 40  0000 C CNN
 F 1 "5K" V 3607 2301 40  0000 C CNN
-F 2 "Resistors_SMD:R_0402_NoSilk" V 3530 2300 30  0001 C CNN
+F 2 "Resistor_SMD:R_0805_2012Metric_Pad1.15x1.40mm_HandSolder" V 3530 2300 30  0001 C CNN
 F 3 "~" H 3600 2300 30  0000 C CNN
 	1    3600 2300
@@
 F 0 "R6" V 7380 2300 40  0000 C CNN
 F 1 "1K" V 7307 2301 40  0000 C CNN
-F 2 "Resistors_THT:R_Axial_DIN0204_L3.6mm_D1.6mm_P7.62mm_Horizontal" V 7230 2300 30  0001 C CNN
+F 2 "Resistor_SMD:R_0805_2012Metric_Pad1.15x1.40mm_HandSolder" V 7230 2300 30  0001 C CNN
 F 3 "~" H 7300 2300 30  0000 C CNN
 	1    7300 2300
@@
 F 0 "R1" V 3030 2300 40  0000 C CNN
 F 1 "5K" V 2957 2301 40  0000 C CNN
-F 2 "Resistors_SMD:R_0402_NoSilk" V 2880 2300 30  0001 C CNN
+F 2 "Resistor_SMD:R_0805_2012Metric_Pad1.15x1.40mm_HandSolder" V 2880 2300 30  0001 C CNN
 F 3 "~" H 2950 2300 30  0000 C CNN
 	1    2950 2300
@@
 F 0 "R3" V 3680 3650 40  0000 C CNN
 F 1 "750" V 3607 3651 40  0000 C CNN
-F 2 "Resistors_THT:R_Axial_DIN0204_L3.6mm_D1.6mm_P7.62mm_Horizontal" V 3530 3650 30  0001 C CNN
+F 2 "Resistor_SMD:R_0805_2012Metric_Pad1.15x1.40mm_HandSolder" V 3530 3650 30  0001 C CNN
 F 3 "~" H 3600 3650 30  0000 C CNN
 	1    3600 3650
@@
 F 0 "U1" H 4200 3450 50  0000 L BNN
 F 1 "ATMEGA8-16AU" H 5450 700 50  0000 L BNN
-F 2 "Housings_QFP:TQFP-32_7x7mm_Pitch0.8mm" H 4950 2250 50  0001 C CIN
+F 2 "Package_DIP:DIP-32_W7.62mm" H 4950 2250 50  0001 C CIN
 F 3 "" H 4950 2250 50  0001 C CNN
 	1    4950 2250
@@
 F 0 "SW1" H 6650 3250 50  0000 L CNN
 F 1 "SW_Push" H 6600 3090 50  0000 C CNN
-F 2 "Buttons_Switches_SMD:SW_SPST_PTS645" H 6600 3350 50  0001 C CNN
+F 2 "Button_Switch_SMD:SW_SPST_PTS645" H 6600 3350 50  0001 C CNN
 F 3 "" H 6600 3350 50  0001 C CNN
 	1    6600 3150
@@
 F 0 "D1" H 3250 1550 50  0000 C CNN
 F 1 "D_Schottky" H 3250 1350 50  0000 C CNN
-F 2 "Diodes_SMD:D_SOT-23_NKA" H 3250 1450 50  0001 C CNN
+F 2 "Diode_SMD:D_SOT-23_NKA" H 3250 1450 50  0001 C CNN
 F 3 "" H 3250 1450 50  0001 C CNN
 	1    3250 1450
@@
 F 0 "D2" H 3250 2150 50  0000 C CNN
 F 1 "D_Schottky" H 3250 1950 50  0000 C CNN
-F 2 "Diodes_SMD:D_SOT-23_NKA" H 3250 2050 50  0001 C CNN
+F 2 "Diode_SMD:D_SOT-23_NKA" H 3250 2050 50  0001 C CNN
 F 3 "" H 3250 2050 50  0001 C CNN
 	1    3250 2050
@@
 F 0 "J1" H 1950 3200 50  0000 C CNN
 F 1 "I_BUTTON" H 2025 2800 50  0000 C CNN
-F 2 "Connectors_Molex:Molex_MicroLatch-53253-0270_02x2.00mm_Straight" H 1950 3100 50  0001 C CNN
+F 2 "Connector_PinHeader_2.54mm:PinHeader_1x02_P2.54mm_Vertical" H 1950 3100 50  0001 C CNN
 F 3 "" H 1950 3100 50  0001 C CNN
 	1    1950 3000
@@
 F 0 "J2" H 2450 3200 50  0000 C CNN
 F 1 "IB_READ" H 2525 2800 50  0000 C CNN
-F 2 "Connectors_Molex:Molex_MicroLatch-53253-0270_02x2.00mm_Straight" H 2450 3100 50  0001 C CNN
+F 2 "Connector_PinHeader_2.54mm:PinHeader_1x02_P2.54mm_Vertical" H 2450 3100 50  0001 C CNN
 F 3 "" H 2450 3100 50  0001 C CNN
 	1    2450 3000
@@
 F 0 "C2" H 5125 6550 50  0000 L CNN
 F 1 "0.1mF" H 5125 6350 50  0000 L CNN
-F 2 "Capacitors_THT:CP_Radial_D5.0mm_P2.50mm" H 5138 6300 50  0001 C CNN
+F 2 "Capacitor_SMD:C_0805_2012Metric_Pad1.15x1.40mm_HandSolder" H 5138 6300 50  0001 C CNN
 F 3 "" H 5100 6450 50  0001 C CNN
 	1    5100 6450
@@
 F 0 "C1" H 3875 1100 50  0000 L CNN
 F 1 "0.1mF" H 3875 900 50  0000 L CNN
-F 2 "Capacitors_THT:CP_Radial_D5.0mm_P2.50mm" H 3888 850 50  0001 C CNN
+F 2 "Capacitor_SMD:C_0805_2012Metric_Pad1.15x1.40mm_HandSolder" H 3888 850 50  0001 C CNN
 F 3 "" H 3850 1000 50  0001 C CNN
 	1    3850 1000
@@
 F 0 "Q2" H 6800 3925 50  0000 L CNN
 F 1 "BC847" H 6800 3850 50  0000 L CNN
-F 2 "TO_SOT_Packages_SMD:SOT-23" H 6800 3775 50  0001 L CIN
+F 2 "Package_TO_SOT_SMD:SOT-23_Handsoldering" H 6800 3775 50  0001 L CIN
 F 3 "" H 6600 3850 50  0001 L CNN
 	1    6600 3850
@@
 F 0 "Q1" H 3650 3150 50  0000 L CNN
 F 1 "BC847" H 3550 2800 50  0000 L CNN
-F 2 "TO_SOT_Packages_SMD:SOT-23" H 4000 2925 50  0001 L CIN
+F 2 "Package_TO_SOT_SMD:SOT-23_Handsoldering" H 4000 2925 50  0001 L CIN
 F 3 "" H 3800 3000 50  0001 L CNN
 	1    3800 3000
@@
 F 0 "J4" H 3650 5850 50  0000 L CNN
 F 1 "USB_OTG" H 3650 5750 50  0000 L CNN
-F 2 "Connectors:USB_Mini-B" H 4000 5350 50  0001 C CNN
+F 2 "Connector_USB:USB_Micro-B_Wuerth_629105150521" H 4000 5350 50  0001 C CNN
 F 3 "" H 4000 5350 50  0001 C CNN
 	1    3850 5400
@@
 F 0 "J3" V 2150 1100 50  0000 C CNN
 F 1 "BATTERY" V 2250 950 50  0000 C CNN
-F 2 "Connectors:bornier2" H 2150 950 50  0001 C CNN
+F 2 "Connector_PinHeader_2.54mm:PinHeader_1x02_P2.54mm_Vertical" H 2150 950 50  0001 C CNN
 F 3 "" H 2150 950 50  0001 C CNN
 	1    2150 950
@@
 F 0 "Y1" H 5850 5700 50  0000 C CNN
 F 1 "12MHz" H 5850 5800 50  0000 C CNN
-F 2 "" H 5850 5900 50  0001 C CNN
+F 2 "Crystal:Crystal_SMD_HC49-SD" H 5850 5900 50  0001 C CNN
 F 3 "~" H 5850 5900 50  0001 C CNN
 	1    5850 5900
@@
 F 0 "C6" H 6165 6296 50  0000 L CNN
 F 1 "22pF" H 6165 6205 50  0000 L CNN
-F 2 "" H 6088 6100 50  0001 C CNN
+F 2 "Capacitor_SMD:C_0805_2012Metric_Pad1.15x1.40mm_HandSolder" H 6088 6100 50  0001 C CNN
 F 3 "~" H 6050 6250 50  0001 C CNN
 	1    6050 6250
@@
 F 0 "C4" H 5715 6296 50  0000 L CNN
 F 1 "22pF" H 5715 6205 50  0000 L CNN
-F 2 "" H 5638 6100 50  0001 C CNN
+F 2 "Capacitor_SMD:C_0805_2012Metric_Pad1.15x1.40mm_HandSolder" H 5638 6100 50  0001 C CNN
 F 3 "~" H 5600 6250 50  0001 C CNN
 	1    5600 6250
@@
 F 0 "C5" H 5915 5046 50  0000 L CNN
 F 1 "0.01uF" H 5915 4955 50  0000 L CNN
-F 2 "" H 5838 4850 50  0001 C CNN
+F 2 "Capacitor_SMD:C_0805_2012Metric_Pad1.15x1.40mm_HandSolder" H 5838 4850 50  0001 C CNN
 F 3 "~" H 5800 5000 50  0001 C CNN
 	1    5800 5000
@@
 F 0 "C3" H 5525 5100 50  0000 L CNN
 F 1 "0.1mF" H 5525 4900 50  0000 L CNN
-F 2 "Capacitors_THT:CP_Radial_D5.0mm_P2.50mm" H 5538 4850 50  0001 C CNN
+F 2 "Capacitor_SMD:C_0805_2012Metric_Pad1.15x1.40mm_HandSolder" H 5538 4850 50  0001 C CNN
 F 3 "" H 5500 5000 50  0001 C CNN
 	1    5500 5000
@@
 F 0 "D3" H 6500 1150 50  0000 C CNN
 F 1 "2^0" H 6500 1250 50  0000 C CNN
-F 2 "" H 6500 1350 50  0001 C CNN
+F 2 "LED_THT:LED_D5.0mm" H 6500 1350 50  0001 C CNN
 F 3 "~" H 6500 1350 50  0001 C CNN
 	1    6500 1350
@@
 F 0 "D5" H 6750 1400 50  0000 C CNN
 F 1 "2^1" H 6750 1500 50  0000 C CNN
-F 2 "" H 6750 1600 50  0001 C CNN
+F 2 "LED_THT:LED_D5.0mm" H 6750 1600 50  0001 C CNN
 F 3 "~" H 6750 1600 50  0001 C CNN
 	1    6750 1600
@@
 P 6500 1850
 F 0 "D4" H 6500 1650 50  0000 C CNN
-F 1 "2^3" H 6500 1750 50  0000 C CNN
-F 2 "" H 6500 1850 50  0001 C CNN
+F 1 "2^2" H 6500 1750 50  0000 C CNN
+F 2 "LED_THT:LED_D5.0mm" H 6500 1850 50  0001 C CNN
 F 3 "~" H 6500 1850 50  0001 C CNN
 	1    6500 1850
@@
 P 6750 2100
 F 0 "D6" H 6750 1900 50  0000 C CNN
-F 1 "2^4" H 6750 2000 50  0000 C CNN
-F 2 "" H 6750 2100 50  0001 C CNN
+F 1 "2^3" H 6750 2000 50  0000 C CNN
+F 2 "LED_THT:LED_D5.0mm" H 6750 2100 50  0001 C CNN
 F 3 "~" H 6750 2100 50  0001 C CNN
 	1    6750 2100
@@
 $EndComp
 Wire Wire Line
-	5950 1350 6350 1350
-Wire Wire Line
 	6650 1350 7300 1350
 Wire Wire Line
@@
 	7300 2100 7300 2150
 Wire Wire Line
-	5950 1450 6350 1450
-Wire Wire Line
-	6350 1450 6350 1600
-Wire Wire Line
-	6350 1600 6600 1600
-Wire Wire Line
-	5950 1550 6300 1550
-Wire Wire Line
-	6300 1550 6300 1850
-Wire Wire Line
 	6300 1850 6350 1850
-Wire Wire Line
-	5950 1650 6250 1650
-Wire Wire Line
-	6250 1650 6250 2100
 Wire Wire Line
 	6250 2100 6600 2100
 NoConn ~ 5950 3250
+NoConn ~ 4150 5600
+NoConn ~ 4050 1550
+NoConn ~ 4050 1650
+NoConn ~ 4050 1250
+NoConn ~ 5950 2650
+NoConn ~ 5950 2550
+NoConn ~ 5950 2450
+NoConn ~ 5950 2350
+NoConn ~ 5950 2250
+NoConn ~ 5950 2150
+NoConn ~ 5950 2050
+NoConn ~ 5950 1950
+NoConn ~ 5950 1750
+Wire Wire Line
+	6350 1350 6150 1350
+Wire Wire Line
+	6150 1350 6150 1650
+Wire Wire Line
+	6150 1650 5950 1650
+Wire Wire Line
+	6600 1600 6050 1600
+Wire Wire Line
+	6050 1600 6050 1550
+Wire Wire Line
+	6050 1550 5950 1550
+Wire Wire Line
+	6300 1450 5950 1450
+Wire Wire Line
+	6300 1450 6300 1850
+Wire Wire Line
+	6250 1300 5950 1300
+Wire Wire Line
+	5950 1300 5950 1350
+Wire Wire Line
+	6250 1300 6250 2100
 $EndSCHEMATC

Commit message: готов прототип печатной платы
Parts:
- removed C2: 0.1mF, Capacitor_SMD:C_0805_2012Metric_Pad1.15x1.40mm_HandSolder, symbol Device:CP
Connections:
- net at D2.2 (A), R4.1: now also C3.1, J4.1 (VBUS), U2.16 (VCC)
Changed lines of the file:
@@
 	3250 2200 3250 4400
-Wire Wire Line
-	3250 4400 5100 4400
 Wire Wire Line
 	5000 3850 4900 3850
@@
 Wire Wire Line
 	5900 4150 6150 4150
-Connection ~ 5100 4400
 Wire Wire Line
 	6100 1000 7850 1000
@@
 Wire Wire Line
 	6200 6650 6200 6850
-Wire Wire Line
-	5100 6650 5100 6600
 $Comp
 L ibutton-rescue:ATMEGA8-16AU U1
@@
 	6700 4150 6600 4150
 $Comp
-L Device:CP C2
-U 1 1 5991EB55
-P 5100 6450
-F 0 "C2" H 5125 6550 50  0000 L CNN
-F 1 "0.1mF" H 5125 6350 50  0000 L CNN
-F 2 "Capacitor_SMD:C_0805_2012Metric_Pad1.15x1.40mm_HandSolder" H 5138 6300 50  0001 C CNN
-F 3 "" H 5100 6450 50  0001 C CNN
-	1    5100 6450
-	1    0    0    -1
-$EndComp
-$Comp
 L Device:CP C1
 U 1 1 5991F2CC
@@
 	3250 1750 3700 1750
 Wire Wire Line
-	5100 4400 5500 4400
-Wire Wire Line
 	7850 2800 7850 2950
 Wire Wire Line
@@
 $EndComp
 Wire Wire Line
-	5100 6650 5600 6650
-Wire Wire Line
 	6050 6100 6050 5900
 Connection ~ 6050 5900
@@
 Wire Wire Line
 	5600 6400 5600 6650
-Connection ~ 5600 6650
 Wire Wire Line
 	5600 6650 6050 6650
@@
 	6400 4800 6400 4900
 Wire Wire Line
-	5100 4400 5100 6300
-Wire Wire Line
-	4150 4700 5500 4700
+	4150 4700 4850 4700
 Wire Wire Line
 	6500 4700 6500 4900
@@
 Wire Wire Line
 	6250 1300 6250 2100
+Wire Wire Line
+	3250 4400 4850 4400
+Wire Wire Line
+	4850 4700 4850 4400
+Connection ~ 4850 4700
+Wire Wire Line
+	4850 4700 5500 4700
+Connection ~ 4850 4400
+Wire Wire Line
+	4850 4400 5500 4400
 $EndSCHEMATC
